File: ee/split_carrier/split_carrier.sch (KiCad schematic (older format))
At the start: 15 parts, among them J1 Conn_01x08, J2 Conn_01x08, J3 Conn_01x08, J4 Conn_01x08, J5 Conn_01x04, J6 STM32F0_Discovery_Header, U2 RC1602A

Commit message: update layout for carrier with new pin assignments
Parts:
- J1, J2, J3, J4: footprint custom:Fan_Controller -> custom:Fan_Controller_all
- J6: symbol STM32F0_Discovery_Header -> STM32F0_Discovery_Header-RESCUE-split_carrier
Connections:
- net +3V3: now also J6.1 (3V), R17.1, R2.1, R2.2, U2.2 (VDD); no longer U2.15 (A/VEE)
- net FAN0_ADC: now also J6.14 (PC3/ADC13); no longer J6.11 (PC0)
- net FAN0_RPM: now also J6.35 (PB13); no longer J6.15 (PA0)
- net FAN1_ADC: now also J6.13 (PC2/ADC12); no longer J6.12 (PC1)
- net FAN1_RPM: now also J6.36 (PB14); no longer J6.16 (PA1)
- net FAN2_ADC: now also J6.12 (PC1/ADC11); no longer J6.13 (PC2)
- net FAN2_RPM: now also J6.63 (PB8); no longer J6.17 (PA2)
- net FAN3_ADC: now also J6.11 (PC0/ADC10); no longer J6.14 (PC3)
- net FAN3_RPM: now also J6.64 (PB9); no longer J6.18 (PA3)
- net GND: now also U2.5 (R/W)
- net LCD_D0: now also J6.15 (PA0); no longer J6.27 (PB0)
- net LCD_D1: now also J6.16 (PA1); no longer J6.28 (PB1)
- net LCD_D2: now also J6.17 (PA2); no longer J6.29 (PB2)
- net LCD_D3: now also J6.18 (PA3); no longer J6.56 (PB3)
- net LCD_D4: now also J6.21 (PA4); no longer J6.57 (PB4)
- net LCD_D5: now also J6.22 (PA5); no longer J6.58 (PB5)
- net LCD_D6: now also J6.23 (PA6); no longer J6.59 (PB6)
- net LCD_D7: now also J6.24 (PA7); no longer J6.60 (PB7)
- net LCD_RS: now also J6.42 (PA8); no longer J6.35 (PB13)
- net FAN4_ADC: now reaches J6.25 (PC4/ADC14)
- net FAN5_ADC: now reaches J6.26 (PC5/ADC15)
- net FAN6_CTRL: now reaches J6.30 (PB10/T2_3)
- net FAN7_CTRL: now reaches J6.31 (PB11/T2_4)
- net UART1_TX: now reaches J6.43 (PA9)
- net UART1_RX: now reaches J6.44 (PA10)
- net SWDIO: now reaches J6.47 (PA13)
- net SWCLK: now reaches J6.50 (PA14)
- net FAN4_CTRL: now reaches J6.51 (T2_1/PA15)
- net at R1.2: now also U2.15 (A/VEE); no longer R2.1
- removed net LCD_RW: J6.36 (PB14), U2.5 (R/W)
- new net FAN5_CTRL: J6.56 (T2_2/PB3)
- new net FAN6_ADC: J6.27 (PB0/ADC8)
- new net FAN7_ADC: J6.28 (PB1/ADC9)
Other:
- moved on the sheet: R1
